File: Hardware/Display/DP_C240_241/schematic-DP_C240_C241/DP_C240_C241.kicad_sch (KiCad schematic)
At the start: 16 parts

Commit message: WIP schematic
Parts:
- D1: renamed from D?; value (none) -> D
- POWER_ON_OFF1: renamed from POWER_ON_OFF; value (none) -> SW_DIP_x01
- R1: renamed from R?; value (none) -> R
- R2, R3, R6: renamed from R?; value (none) -> 500
- R8: renamed from R?; value (none) -> 1500
- Rfb1, Rfb2: renamed from R?; value 1500 -> (none)
- motor1: renamed from motor; value (none) -> Conn_01x05
- remote_keypad1: renamed from remote_keypad; value (none) -> Conn_01x06
- gave numbers to parts that had none: 4
- renumbered DOWN to DOWN1

Commit message: WIP schematic
Parts:
- R7: value 500 -> (none)
- R8: value 1500 -> (none)
- Rfb1, Rfb2: value (none) -> ??
- renumbered DOWN1 to DOWN, POWER_ON_OFF1 to POWER_ONOFF
Connections:
- net microcontroller_remote_ONOFF: now reaches D1.2 (A), R1.2
- net microcontroller_remote_DOWN: now reaches D2.2 (A), R4.2
Other:
- moved on the sheet: D1, D2, DOWN, POWER_ONOFF, R1, R2, R3, R4, R5, R6, R7, R8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
